Commit message: Create a new env and install the mask effector

File: assistive_gym/envs/assets/jaco/j2s7s300_gym.urdf (robot description, URDF)
Before this commit: robot j2s7s300, 16 links, 15 joints
Links:
- removed link j2s7s300_link_finger_1
- removed link j2s7s300_link_finger_2
- removed link j2s7s300_link_finger_3
- removed link j2s7s300_link_finger_tip_1
- removed link j2s7s300_link_finger_tip_2
- removed link j2s7s300_link_finger_tip_3
- link j2s7s300_link_7: geometry collision mesh filename=meshes/mask_effector.STL; visual mesh filename=meshes/mask_effector.STL
Joints:
- removed joint j2s7s300_joint_finger_1
- removed joint j2s7s300_joint_finger_2
- removed joint j2s7s300_joint_finger_3
- removed joint j2s7s300_joint_finger_tip_1
- removed joint j2s7s300_joint_finger_tip_2
- removed joint j2s7s300_joint_finger_tip_3

Commit message: Update j2s7s300_gym.urdf

File: assistive_gym/envs/assets/jaco/j2s7s300_gym.urdf (robot description, URDF)
Before this commit: robot j2s7s300, 10 links, 9 joints
Links:
- link j2s7s300_link_7: mass 0.99 -> 0.234257

Commit message: Update the mask effector

File: assistive_gym/envs/assets/jaco/j2s7s300_gym.urdf (robot description, URDF)
Before this commit: robot j2s7s300, 10 links, 9 joints
Links:
- removed link j2s7s300_link_7
- added link j2s7s300_mask; collision mesh filename=meshes/mask.STL; visual mesh filename=meshes/mask.STL
- added link j2s7s300_mask_holder, mass 0.161340; collision mesh filename=meshes/mask_holder.STL; visual mesh filename=meshes/mask_holder.STL
- link j2s7s300_end_effector: geometry collision box size=0 0 0; visual box size=0.01 0.01 0.01
Joints:
- added joint j2s7s300_joint_8: type fixed, parent j2s7s300_mask_holder, child j2s7s300_mask, origin xyz=0 0 0 rpy=0 0 0, axis 0 0 0
- joint j2s7s300_joint_7: child j2s7s300_link_7 -> j2s7s300_mask_holder
- joint j2s7s300_joint_end_effector: limit lower=0 upper=0 effort=2000 velocity=1 -> (none); origin xyz=0 0 -0.1600 rpy=3.14159265359 0 0 -> xyz=0 0 -0.165 rpy=3.14159265359 0 0; parent j2s7s300_link_7 -> j2s7s300_mask

Commit message: Update the mask effector

File: assistive_gym/envs/assets/jaco/j2s7s300_gym.urdf (robot description, URDF)
Before this commit: robot j2s7s300, 11 links, 10 joints
Joints:
- joint j2s7s300_joint_end_effector: parent j2s7s300_mask -> j2s7s300_mask_holder

Commit message: Reoriented mask holder end effector and modified robot arm starting position

File: assistive_gym/envs/assets/jaco/j2s7s300_gym.urdf (robot description, URDF)
Before this commit: robot j2s7s300, 11 links, 10 joints
Joints:
- joint j2s7s300_joint_end_effector: origin xyz=0 0 -0.165 rpy=3.14159265359 0 0 -> xyz=0 0 -0.165 rpy=4.71238898039 0 0

Commit message: Updated the end effector

File: assistive_gym/envs/assets/jaco/j2s7s300_gym.urdf (robot description, URDF)
Before this commit: robot j2s7s300, 11 links, 10 joints
Links:
- added link j2s7s300_camera; collision mesh filename=meshes/camera.STL; visual mesh filename=meshes/camera.STL
Joints:
- added joint j2s7s300_joint_9: type fixed, parent j2s7s300_mask_holder, child j2s7s300_camera, origin xyz=0 0 0 rpy=0 0 0, axis 0 0 0

Commit message: Changed the design back

File: assistive_gym/envs/assets/jaco/j2s7s300_gym.urdf (robot description, URDF)
Before this commit: robot j2s7s300, 12 links, 11 joints
Links:
- removed link j2s7s300_camera
Joints:
- removed joint j2s7s300_joint_9
